File: electronics/controller/controller.kicad_pcb (KiCad board)
At the start: 2 copper layers, 55 parts, among them J1 AZ_STEPPER_TEMP, J10 USB C, J11 PWR IN, J2 EL_STEPPER_TEMP, J3 TEMP_PROBE, J4 I2C, J5 AZ_ENDSTOP, J6 UART, J7 EL_ENDSTOP1, J8 EL_SERVO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

Commit message: lol
Parts:
- added C14: 47u, Capacitor_SMD:CP_Elec_8x10, F.Cu at (115.8, 179.1)
- added C16: 47u, Capacitor_SMD:CP_Elec_8x10, F.Cu at (146.9, 172.6)
- added C18: 150u, Capacitor_SMD:CP_Elec_10x10, F.Cu at (103.0, 180.1)
- added C20: 150u, Capacitor_SMD:CP_Elec_10x10, F.Cu at (134.1, 175.6)
- added D3: SS36, Diode_SMD:D_SMA, F.Cu at (148.2, 187.7)
- added H1: Mount, MountingHole:MountingHole_2.7mm_M2.5_DIN965_Pad, F.Cu at (87.0, 52.0)
- added H2: Mount, MountingHole:MountingHole_2.7mm_M2.5_DIN965_Pad, F.Cu at (213.0, 110.5)
- added H3: Mount, MountingHole:MountingHole_2.7mm_M2.5_DIN965_Pad, F.Cu at (213.0, 116.8)
- added H4: Mount, MountingHole:MountingHole_2.7mm_M2.5_DIN965_Pad, F.Cu at (213.0, 123.0)
- added L1: 68u, Inductor_SMD:L_Coilcraft_MSS1260-XXX, F.Cu at (133.8, 188.5)
- added U4: LM2596S-3.3, Package_TO_SOT_SMD:TO-263-5_TabPin3, F.Cu at (54.4, 140.6)
- C15, C17, C19, C21: footprint Capacitor_SMD:C_0805_2012Metric -> Capacitor_SMD:C_1210_3225Metric
- moved J6 108.2 mm to (83.9, 118.6)
- moved U4 94.7 mm to (74.7, 155.1)
- moved J9 82.8 mm to (104.5, 142.4)
- moved J7 80.7 mm to (194.7, 68.8)
- moved D1 78.4 mm to (96.4, 116.9)
- moved C6 76.8 mm to (84.0, 112.7)
- moved C4 74.3 mm to (86.2, 112.7), turned to 180 degrees
- moved C2 74.1 mm to (87.7, 73.0), turned to -90 degrees
- moved J5 70.5 mm to (198.2, 80.3)
- moved R8 65.5 mm to (84.2, 142.1)
- moved D2 65.3 mm to (96.3, 135.6), turned to 180 degrees
- moved SW3 64.2 mm to (100.3, 80.3), turned to 90 degrees
- moved C5 63.4 mm to (87.7, 60.7), turned to 180 degrees
- moved J8 59.2 mm to (215.7, 138.4)
- moved R1 59.2 mm to (206.1, 139.1)
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- renumbered J9 to J10, J10 to J11, J11 to J9
Connections:
- C15 pad 1: +3V3 -> VCC
- C17 pad 1: VCC -> +3V3
- C19 pad 1: +3V3 -> VCC
- C21 pad 1: VCC -> +3V3
- M1 pad 1: Net-(A1-A1) -> Net-(A1-A2)
- M1 pad 2: Net-(A1-A2) -> Net-(A1-A1)
- M2 pad 1: Net-(A2-A1) -> Net-(A2-A2)
- M2 pad 2: Net-(A2-A2) -> Net-(A2-A1)
Routing:
- net /~{AZ_FAULT}: track 0.00 -> 19.4 mm
- net Net-(A1-B2): track 0.00 -> 10.3 mm
- net Net-(A1-A2): track 0.00 -> 10.1 mm
- net Net-(A1-B1): track 0.00 -> 9.29 mm
- net Net-(A1-A1): track 0.00 -> 9.13 mm
- net /CC1: track 0.00 -> 6.07 mm
- net /CC2: track 0.00 -> 5.78 mm
- added copper zone on B.Cu, net GND
- added copper zone on F.Cu, net GND
- added copper zone on F.Cu, net VCC
Other:
- board outline added: 100 x 100 mm
